Commit message: car and teleoperation

File: urdf/car.xacro (robot description, xacro)
@@ -19,10 +19,10 @@
   <xacro:property name="Iz_wheel" value="${0.5*wheel_mass*wheel_link_radius*wheel_link_radius}"/>
   <xacro:property name="I_wheel" value="${(1.0/12.0) * wheel_mass * (3.0 * wheel_link_radius*wheel_link_radius+wheel_link_length*wheel_link_length)}"/>
-  <xacro:macro name="interia_wheel">
-        <intertial>
+  <xacro:macro name="inertia_wheel">
+        <inertial>
         <origin rpy="0 0 0" xyz="0 0 0"/>
         <mass value="${wheel_mass}"/>
-        <interia ixx="${I_wheel}" ixy="0.0" ixz="0.0" iyy="${I_wheel}" iyz="0" izz="${Iz_wheel}"/>
-        </intertial>
+        <inertia ixx="${I_wheel}" ixy="0.0" ixz="0.0" iyy="${I_wheel}" iyz="0" izz="${Iz_wheel}"/>
+        </inertial>
   </xacro:macro>
   <xacro:include filename="$(find ee148_project)/urdf/robot.gazebo"/>
@@ -50,5 +50,5 @@
             <origin rpy="0 0 0" xyz="0 0 0"/>
             <mass value="${body_mass}"/>
-            <intertia
+            <inertia
             ixx="${(1/12) * body_mass*(body_link_y_dim*body_link_y_dim+body_link_z_dim*body_link_z_dim)}" ixy="0"
             ixz="0" iyy="${(1/12)*body_mass*(body_link_x_dim*body_link_x_dim+body_link_z_dim*body_link_z_dim)}"
@@ -79,5 +79,5 @@
                 </geometry>
         </collision>
-        <xacro:interia_wheel />
+        <xacro:inertia_wheel />
 </link>
 <!-- Back left wheen and joint-->
@@ -103,5 +103,5 @@
                 </geometry>
         </collision>
-        <xacro:interia_wheel />
+        <xacro:inertia_wheel />
 </link>
 <!--Front right wheel and joint-->
@@ -127,5 +127,5 @@
                 </geometry>
         </collision>
-        <xacro:interia_wheel />
+        <xacro:inertia_wheel />
 </link>
 <!--Front left wheel and joint-->
@@ -151,5 +151,5 @@
                 </geometry>
         </collision>
-        <xacro:interia_wheel />
+        <xacro:inertia_wheel />
 </link>
 </robot>

Commit message: fixed synch issues

File: urdf/car.xacro (robot description, xacro)
@@ -1,4 +1,11 @@
 <?xml version="1.0"?>
-<robot xmlns:xacro="http://www.ros.org/wiki/xacro" name="simple_ackermann_car">
+<robot xmlns:xacro="http://www.ros.org/wiki/xacro" name="robot">
+  <xacro:include filename="$(find ee148_project)/urdf/gazebo_control.xacro" />
+<material name = "yellow">
+        <color rgba = "1 1 0 1" />
+ </material>
+ <material name = "red">
+        <color rgba = "1 0 0 1" />
+ </material>
   <!-- Define parameters for size and position -->
   <xacro:property name="body_link_x_dim" value="1.0" />
@@ -26,12 +33,13 @@
         </inertial>
   </xacro:macro>
-  <xacro:include filename="$(find ee148_project)/urdf/robot.gazebo"/>
-  <link name = "dummy">
+  <!--xacro:include filename="$(find ee148_project)/urdf/gazebo_control.xacro"-/ -->
+  <link name = "base_link">
   </link>
-  <joint name="dummy joint" type="fixed">
-        <parent link="dummy"/>
+  <!--BODY LINK-->
+<joint name="body_joint" type="fixed">
+        <parent link="base_link"/>
         <child link="body_link"/>
-  </joint>
-  <!--BODY LINK-->
+        <origin xyz = "0 0 0.35"/>
+</joint>
 <link name="body_link">
   <visual>
@@ -40,4 +48,5 @@
           </geometry>
           <origin rpy="0 0 0" xyz="0 0 0"/>
+          <material name = "red"/>
   </visual>
   <collision>
@@ -57,4 +66,7 @@
         </inertial>
 </link>
+    <gazebo reference="body_link">
+        <material>Gazebo/Red</material>
+    </gazebo>
 <!-- Back right wheel and joint-->
 <joint name ="wheel1_joint" type="continuous" >
@@ -72,4 +84,5 @@
                 <cylinder length="${wheel_link_length}" radius="${wheel_link_radius}" />
             </geometry>
+            <material name = "yellow"/>
         </visual>
         <collision>
@@ -81,4 +94,7 @@
         <xacro:inertia_wheel />
 </link>
+    <gazebo reference="wheel1_link">
+        <material>Gazebo/Yellow</material>
+    </gazebo>
 <!-- Back left wheen and joint-->
 <joint name ="wheel2_joint" type="continuous" >
@@ -96,4 +112,5 @@
                 <cylinder length="${wheel_link_length}" radius="${wheel_link_radius}" />
             </geometry>
+            <material name = "yellow"/>
         </visual>
         <collision>
@@ -105,4 +122,7 @@
         <xacro:inertia_wheel />
 </link>
+    <gazebo reference="wheel2_link">
+        <material>Gazebo/Yellow</material>
+    </gazebo>
 <!--Front right wheel and joint-->
 <joint name ="wheel3_joint" type="continuous" >
@@ -120,4 +140,5 @@
                 <cylinder length="${wheel_link_length}" radius="${wheel_link_radius}" />
             </geometry>
+            <material name = "yellow"/>
         </visual>
         <collision>
@@ -129,4 +150,7 @@
         <xacro:inertia_wheel />
 </link>
+    <gazebo reference="wheel3_link">
+        <material>Gazebo/Yellow</material>
+    </gazebo>
 <!--Front left wheel and joint-->
 <joint name ="wheel4_joint" type="continuous" >
@@ -144,4 +168,5 @@
                 <cylinder length="${wheel_link_length}" radius="${wheel_link_radius}" />
             </geometry>
+            <material name = "yellow"/>
         </visual>
         <collision>
@@ -153,3 +178,6 @@
         <xacro:inertia_wheel />
 </link>
+    <gazebo reference="wheel4_link">
+        <material>Gazebo/Yellow</material>
+    </gazebo>
 </robot>
