Commit message: scan topic published

File: urdf/car.urdf.xacro (robot description, xacro)
@@ -1,5 +1,5 @@
 <?xml version="1.0"?>
 <robot xmlns:xacro="http://www.ros.org/wiki/xacro" name="robot">
-<xacro:include filename="$(find ee148_project)/urdf/car.xacro" />
-<xacro:include filename="$(find ee148_project)/urdf/lidar.xacro" />
+    <xacro:include filename="$(find ee148_project)/urdf/car.xacro" />
+    <xacro:include filename="$(find ee148_project)/urdf/lidar.xacro" />
 </robot>

File: urdf/car.xacro (robot description, xacro)
@@ -1,5 +1,4 @@
 <?xml version="1.0"?>
 <robot xmlns:xacro="http://www.ros.org/wiki/xacro" name="robot">
-  <xacro:include filename="$(find ee148_project)/urdf/gazebo_control.xacro" />
 <material name = "yellow">
         <color rgba = "1 1 0 1" />
@@ -68,4 +67,6 @@
     <gazebo reference="body_link">
         <material>Gazebo/Red</material>
+        <mu1>0.2</mu1>
+        <mu2>0.2</mu2>
     </gazebo>
 <!-- Back right wheel and joint-->
@@ -96,4 +97,6 @@
     <gazebo reference="wheel1_link">
         <material>Gazebo/Yellow</material>
+        <mu1>0.2</mu1>
+        <mu2>0.2</mu2>
     </gazebo>
 <!-- Back left wheen and joint-->
@@ -124,4 +127,6 @@
     <gazebo reference="wheel2_link">
         <material>Gazebo/Yellow</material>
+        <mu1>0.2</mu1>
+        <mu2>0.2</mu2>
     </gazebo>
 <!--Front right wheel and joint-->
@@ -152,4 +157,6 @@
     <gazebo reference="wheel3_link">
         <material>Gazebo/Yellow</material>
+        <mu1>0.2</mu1>
+        <mu2>0.2</mu2>
     </gazebo>
 <!--Front left wheel and joint-->
@@ -180,4 +187,8 @@
     <gazebo reference="wheel4_link">
         <material>Gazebo/Yellow</material>
+        <mu1>0.2</mu1>
+        <mu2>0.2</mu2>
     </gazebo>
+      <xacro:include filename="$(find ee148_project)/urdf/gazebo_control.xacro" />
+  <!-- <xacro:include filename="$(find ee148_project)/urdf/lidar.xacro" /> -->
 </robot>

File: urdf/gazebo_control.xacro (robot description, xacro)
@@ -3,4 +3,5 @@
     <gazebo>
         <plugin name="skid_steer_drive_controller" filename="libgazebo_ros_skid_steer_drive.so">
+            <updateRate>100.0</updateRate>
             <!-- Wheel Information -->
             <leftFrontJoint>wheel4_joint</leftFrontJoint>
@@ -8,6 +9,7 @@
             <leftRearJoint>wheel2_joint</leftRearJoint>
             <rightRearJoint>wheel1_joint</rightRearJoint>
-            <wheelSeparation>0.297</wheelSeparation>
-            <wheelDiameter>0.066</wheelDiameter>
+            <wheelSeparation>0.7</wheelSeparation>
+            <wheelDiameter>0.3</wheelDiameter>
+            <torque>1000</torque>
         <!-- Command and Odometry Topics -->
             <commandTopic>cmd_vel</commandTopic>
@@ -17,5 +19,7 @@
             <robotBaseFrame>base_link</robotBaseFrame>
             <broadcastTF>true</broadcastTF>
-            <publishOdomTf>true</publishOdomTf>
+            <publishOdom>true</publishOdom>
+            <publishWheelTF>true</publishWheelTF>
+            <publishWheelJointState>true</publishWheelJointState>
             <covariance_x>0.0001</covariance_x>
             <covariance_y>0.0001</covariance_y>

File: urdf/lidar.xacro (robot description, xacro)
@@ -4,5 +4,5 @@
         <color rgba = "0.1 0.1 1 1" />
  </material>
-    <joint name="last_joint" type="fixed">
+    <joint name="laser_joint" type="fixed">
         <parent link="body_link"/>
         <child link="laser_frame"/>
@@ -45,10 +45,7 @@
                 </range>
             </ray>
-            <plugin name="laser_controller" filename="libgazebo_ros_ray_sensor.so">
-                <ros>
-                    <argument>~/out:=scan</argument>
-                </ros>
-                <output_type>sensor_msgs/LaserScan</output_type>
-                <frame_name>laser_frame</frame_name>
+            <plugin name="laser_controller" filename="libgazebo_ros_laser.so">
+                <topicName>/scan</topicName>
+                <frameName>laser_frame</frameName>
             </plugin>
         </sensor>
